Commit message: refine Lift2 collision sphere calibration

File: maniskill_curobo_fangzhou/generated/lift2_maniskill_collision_spheres.urdf (robot description, URDF)
Before this commit: robot lift2, 21 links, 20 joints
Links:
- link left_link16: geometry collision sphere radius=0.006; collision sphere radius=0.018
- link left_link17: geometry collision sphere radius=0.012; collision sphere radius=0.012
- link left_link18: geometry collision sphere radius=0.01; collision sphere radius=0.01
- link right_link22: geometry collision sphere radius=0.035; collision sphere radius=0.035
- link right_link23: geometry collision sphere radius=0.022; collision sphere radius=0.025
- link right_link24: geometry collision sphere radius=0.034; collision sphere radius=0.034
- link right_link25: geometry collision sphere radius=0.031; collision sphere radius=0.031
- link right_link26: geometry collision sphere radius=0.006; collision sphere radius=0.018
- link right_link27: geometry collision sphere radius=0.012; collision sphere radius=0.012
- link right_link28: geometry collision sphere radius=0.01; collision sphere radius=0.01

File: maniskill_curobo_fangzhou/generated/lift2_maniskill_collision_spheres_debug.urdf (robot description, URDF)
Before this commit: robot lift2, 21 links, 20 joints
Links:
- link left_link11: geometry collision sphere radius=0.058; visual mesh filename=/home/openclaw-server/projects/zerograsp/maniskill_curobo_f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
- link left_link12: geometry collision sphere radius=0.043728; collision sphere radius=0.0456612
- link left_link13: geometry collision sphere radius=0.0191721; collision sphere radius=0.0196326
- link left_link14: geometry collision sphere radius=0.0450891; collision sphere radius=0.0478864
- link left_link15: geometry collision sphere radius=0.0340497; collision sphere radius=0.0374199
- link left_link16: geometry collision sphere radius=0.006; collision sphere radius=0.018
- link left_link17: geometry collision sphere radius=0.012; collision sphere radius=0.012
- link left_link18: geometry collision sphere radius=0.01; collision sphere radius=0.01
- link right_link21: geometry collision sphere radius=0.058; visual mesh filename=/home/openclaw-server/projects/zerograsp/maniskill_curobo_f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
- link right_link22: geometry collision sphere radius=0.035; collision sphere radius=0.035
- link right_link23: geometry collision sphere radius=0.022; collision sphere radius=0.025
- link right_link24: geometry collision sphere radius=0.034; collision sphere radius=0.034
- link right_link25: geometry collision sphere radius=0.031; collision sphere radius=0.031
- link right_link26: geometry collision sphere radius=0.006; collision sphere radius=0.018
- link right_link27: geometry collision sphere radius=0.012; collision sphere radius=0.012
- link right_link28: geometry collision sphere radius=0.01; collision sphere radius=0.01

Commit message: Add Lift2 M4C execution diagnostics

File: maniskill_curobo_fangzhou/generated/lift2_maniskill_collision_spheres.urdf (robot description, URDF)
Before this commit: robot lift2, 21 links, 20 joints
Links:
- added link head_camera_link
- added link right_tcp
Joints:
- added joint head_camera_fixed_joint: type fixed, parent base_link, child head_camera_link, origin xyz=0.30000001192092896 0.0 1.041599988937378 rpy=0.0 0.7611162950495652 0.0
- added joint right_tcp_fixed_joint: type fixed, parent right_link26, child right_tcp, origin xyz=0.14496999979019165 0.0017859999788925052 0.0 rpy=0.0 0.0 0.0

File: maniskill_curobo_fangzhou/generated/lift2_maniskill_collision_spheres_debug.urdf (robot description, URDF)
Before this commit: robot lift2, 21 links, 20 joints
Links:
- added link head_camera_link
- added link right_tcp
Joints:
- added joint head_camera_fixed_joint: type fixed, parent base_link, child head_camera_link, origin xyz=0.30000001192092896 0.0 1.041599988937378 rpy=0.0 0.7611162950495652 0.0
- added joint right_tcp_fixed_joint: type fixed, parent right_link26, child right_tcp, origin xyz=0.14496999979019165 0.0017859999788925052 0.0 rpy=0.0 0.0 0.0

File: maniskill_curobo_fangzhou/generated/lift2_maniskill_full_collision.urdf (robot description, URDF)
Before this commit: robot lift2, 22 links, 21 joints
Links:
- added link right_tcp
- link base_link: geometry collision mesh filename=/home/openclaw-server/projects/zerograsp/maniskill_curobo_f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; visual mesh filename=/home/openclaw-server/projects/zerograsp/maniskill_curobo_f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
- link body4: geometry collision mesh filename=/home/openclaw-server/projects/zerograsp/maniskill_curobo_f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; visual mesh filename=/home/openclaw-server/projects/zerograsp/maniskill_curobo_f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
- link left_link11: geometry collision mesh filename=/home/openclaw-server/projects/zerograsp/maniskill_curobo_f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; visual mesh filename=/home/openclaw-server/projects/zerograsp/maniskill_curobo_f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
- link left_link12: geometry collision mesh filename=/home/openclaw-server/projects/zerograsp/maniskill_curobo_f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; visual mesh filename=/home/openclaw-server/projects/zerograsp/maniskill_curobo_f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
- link left_link13: geometry collision mesh filename=/home/openclaw-server/projects/zerograsp/maniskill_curobo_f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; visual mesh filename=/home/openclaw-server/projects/zerograsp/maniskill_curobo_f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
- link left_link14: geometry collision mesh filename=/home/openclaw-server/projects/zerograsp/maniskill_curobo_f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; visual mesh filename=/home/openclaw-server/projects/zerograsp/maniskill_curobo_f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
- link left_link15: geometry collision mesh filename=/home/openclaw-server/projects/zerograsp/maniskill_curobo_f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; visual mesh filename=/home/openclaw-server/projects/zerograsp/maniskill_curobo_f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
- link left_link16: geometry collision mesh filename=/home/openclaw-server/projects/zerograsp/maniskill_curobo_f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; visual mesh filename=/home/openclaw-server/projects/zerograsp/maniskill_curobo_f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
- link left_link17: geometry collision mesh filename=/home/openclaw-server/projects/zerograsp/maniskill_curobo_f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; visual mesh filename=/home/openclaw-server/projects/zerograsp/maniskill_curobo_f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
- link left_link18: geometry collision mesh filename=/home/openclaw-server/projects/zerograsp/maniskill_curobo_f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; visual mesh filename=/home/openclaw-server/projects/zerograsp/maniskill_curobo_f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
- link right_link21: geometry collision mesh filename=/home/openclaw-server/projects/zerograsp/maniskill_curobo_f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; visual mesh filename=/home/openclaw-server/projects/zerograsp/maniskill_curobo_f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
- link right_link22: geometry collision mesh filename=/home/openclaw-server/projects/zerograsp/maniskill_curobo_f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; visual mesh filename=/home/openclaw-server/projects/zerograsp/maniskill_curobo_f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
- link right_link23: geometry collision mesh filename=/home/openclaw-server/projects/zerograsp/maniskill_curobo_f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; visual mesh filename=/home/openclaw-server/projects/zerograsp/maniskill_curobo_f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
- link right_link24: geometry collision mesh filename=/home/openclaw-server/projects/zerograsp/maniskill_curobo_f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; visual mesh filename=/home/openclaw-server/projects/zerograsp/maniskill_curobo_f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
- link right_link25: geometry collision mesh filename=/home/openclaw-server/projects/zerograsp/maniskill_curobo_f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; visual mesh filename=/home/openclaw-server/projects/zerograsp/maniskill_curobo_f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
- link right_link26: geometry collision mesh filename=/home/openclaw-server/projects/zerograsp/maniskill_curobo_f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; visual mesh filename=/home/openclaw-server/projects/zerograsp/maniskill_curobo_f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
- link right_link27: geometry collision mesh filename=/home/openclaw-server/projects/zerograsp/maniskill_curobo_f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; visual mesh filename=/home/openclaw-server/projects/zerograsp/maniskill_curobo_f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
- link right_link28: geometry collision mesh filename=/home/openclaw-server/projects/zerograsp/maniskill_curobo_f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; visual mesh filename=/home/openclaw-server/projects/zerograsp/maniskill_curobo_f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
- link wheel1: geometry collision mesh filename=/home/openclaw-server/projects/zerograsp/maniskill_curobo_f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; visual mesh filename=/home/openclaw-server/projects/zerograsp/maniskill_curobo_f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
- link wheel2: geometry collision mesh filename=/home/openclaw-server/projects/zerograsp/maniskill_curobo_f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; visual mesh filename=/home/openclaw-server/projects/zerograsp/maniskill_curobo_f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
- link wheel3: geometry collision mesh filename=/home/openclaw-server/projects/zerograsp/maniskill_curobo_f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; visual mesh filename=/home/openclaw-server/projects/zerograsp/maniskill_curobo_f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
Joints:
- added joint right_tcp_fixed_joint: type fixed, parent right_link26, child right_tcp, origin xyz=0.14496999979019165 0.0017859999788925052 0.0 rpy=0.0 0.0 0.0
