Commit message: Prepare GitHub sync without large artifacts

File: maniskill_curobo_fangzhou/generated/lift2_maniskill_collision_spheres.urdf (robot description, URDF)
Before this commit: robot lift2, 23 links, 22 joints
Links:
- link base_link: geometry visual mesh filename=/home/xufangjin/workspace/zerograsp/maniskill_curobo_fangzh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
- link body4: geometry visual mesh filename=/home/xufangjin/workspace/zerograsp/maniskill_curobo_fangzh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
- link left_link11: geometry collision sphere radius=0.058; visual mesh filename=/home/xufangjin/workspace/zerograsp/maniskill_curobo_fangzh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
- link left_link12: geometry collision sphere radius=0.043728; collision sphere radius=0.0456612
- link left_link13: geometry collision sphere radius=0.0191721; collision sphere radius=0.0196326
- link left_link14: geometry collision sphere radius=0.0450891; collision sphere radius=0.0478864
- link left_link15: geometry collision sphere radius=0.0340497; collision sphere radius=0.0374199
- link left_link16: geometry collision sphere radius=0.006; collision sphere radius=0.018
- link left_link17: geometry collision sphere radius=0.012; collision sphere radius=0.012
- link left_link18: geometry collision sphere radius=0.01; collision sphere radius=0.01
- link right_link21: geometry collision sphere radius=0.058; visual mesh filename=/home/xufangjin/workspace/zerograsp/maniskill_curobo_fangzh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
- link right_link22: geometry collision sphere radius=0.035; collision sphere radius=0.035
- link right_link23: geometry collision sphere radius=0.022; collision sphere radius=0.025
- link right_link24: geometry collision sphere radius=0.034; collision sphere radius=0.034
- link right_link25: geometry collision sphere radius=0.031; collision sphere radius=0.031
- link right_link26: geometry collision sphere radius=0.006; collision sphere radius=0.018
- link right_link27: geometry collision sphere radius=0.012; collision sphere radius=0.012
- link right_link28: geometry collision sphere radius=0.01; collision sphere radius=0.01
- link wheel1: geometry visual mesh filename=/home/xufangjin/workspace/zerograsp/maniskill_curobo_fangzh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
- link wheel2: geometry visual mesh filename=/home/xufangjin/workspace/zerograsp/maniskill_curobo_fangzh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
- link wheel3: geometry visual mesh filename=/home/xufangjin/workspace/zerograsp/maniskill_curobo_fangzh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

File: maniskill_curobo_fangzhou/generated/lift2_maniskill_collision_spheres_debug.urdf (robot description, URDF)
Before this commit: robot lift2, 23 links, 22 joints
Links:
- link base_link: geometry visual mesh filename=/home/xufangjin/workspace/zerograsp/maniskill_curobo_fangzh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
- link body4: geometry visual mesh filename=/home/xufangjin/workspace/zerograsp/maniskill_curobo_fangzh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
- link left_link11: geometry collision sphere radius=0.058; visual mesh filename=/home/xufangjin/workspace/zerograsp/maniskill_curobo_fangzh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
- link left_link12: geometry collision sphere radius=0.043728; collision sphere radius=0.0456612
- link left_link13: geometry collision sphere radius=0.0191721; collision sphere radius=0.0196326
- link left_link14: geometry collision sphere radius=0.0450891; collision sphere radius=0.0478864
- link left_link15: geometry collision sphere radius=0.0340497; collision sphere radius=0.0374199
- link left_link16: geometry collision sphere radius=0.006; collision sphere radius=0.018
- link left_link17: geometry collision sphere radius=0.012; collision sphere radius=0.012
- link left_link18: geometry collision sphere radius=0.01; collision sphere radius=0.01
- link right_link21: geometry collision sphere radius=0.058; visual mesh filename=/home/xufangjin/workspace/zerograsp/maniskill_curobo_fangzh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
- link right_link22: geometry collision sphere radius=0.035; collision sphere radius=0.035
- link right_link23: geometry collision sphere radius=0.022; collision sphere radius=0.025
- link right_link24: geometry collision sphere radius=0.034; collision sphere radius=0.034
- link right_link25: geometry collision sphere radius=0.031; collision sphere radius=0.031
- link right_link26: geometry collision sphere radius=0.006; collision sphere radius=0.018
- link right_link27: geometry collision sphere radius=0.012; collision sphere radius=0.012
- link right_link28: geometry collision sphere radius=0.01; collision sphere radius=0.01
- link wheel1: geometry visual mesh filename=/home/xufangjin/workspace/zerograsp/maniskill_curobo_fangzh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
- link wheel2: geometry visual mesh filename=/home/xufangjin/workspace/zerograsp/maniskill_curobo_fangzh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
- link wheel3: geometry visual mesh filename=/home/xufangjin/workspace/zerograsp/maniskill_curobo_fangzh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

File: maniskill_curobo_fangzhou/generated/lift2_maniskill_full_collision.urdf (robot description, URDF)
Before this commit: robot lift2, 23 links, 22 joints
Links:
- link base_link: geometry collision mesh filename=/home/xufangjin/workspace/zerograsp/maniskill_curobo_fangzh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; visual mesh filename=/home/xufangjin/workspace/zerograsp/maniskill_curobo_fangzh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
- link body4: geometry collision mesh filename=/home/xufangjin/workspace/zerograsp/maniskill_curobo_fangzh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; visual mesh filename=/home/xufangjin/workspace/zerograsp/maniskill_curobo_fangzh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
- link left_link11: geometry collision mesh filename=/home/xufangjin/workspace/zerograsp/maniskill_curobo_fangzh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; visual mesh filename=/home/xufangjin/workspace/zerograsp/maniskill_curobo_fangzh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
- link left_link12: geometry collision mesh filename=/home/xufangjin/workspace/zerograsp/maniskill_curobo_fangzh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; visual mesh filename=/home/xufangjin/workspace/zerograsp/maniskill_curobo_fangzh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
- link left_link13: geometry collision mesh filename=/home/xufangjin/workspace/zerograsp/maniskill_curobo_fangzh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; visual mesh filename=/home/xufangjin/workspace/zerograsp/maniskill_curobo_fangzh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
- link left_link14: geometry collision mesh filename=/home/xufangjin/workspace/zerograsp/maniskill_curobo_fangzh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; visual mesh filename=/home/xufangjin/workspace/zerograsp/maniskill_curobo_fangzh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
- link left_link15: geometry collision mesh filename=/home/xufangjin/workspace/zerograsp/maniskill_curobo_fangzh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; visual mesh filename=/home/xufangjin/workspace/zerograsp/maniskill_curobo_fangzh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
- link left_link16: geometry collision mesh filename=/home/xufangjin/workspace/zerograsp/maniskill_curobo_fangzh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; visual mesh filename=/home/xufangjin/workspace/zerograsp/maniskill_curobo_fangzh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
- link left_link17: geometry collision mesh filename=/home/xufangjin/workspace/zerograsp/maniskill_curobo_fangzh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; visual mesh filename=/home/xufangjin/workspace/zerograsp/maniskill_curobo_fangzh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
- link left_link18: geometry collision mesh filename=/home/xufangjin/workspace/zerograsp/maniskill_curobo_fangzh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; visual mesh filename=/home/xufangjin/workspace/zerograsp/maniskill_curobo_fangzh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
- link right_link21: geometry collision mesh filename=/home/xufangjin/workspace/zerograsp/maniskill_curobo_fangzh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; visual mesh filename=/home/xufangjin/workspace/zerograsp/maniskill_curobo_fangzh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
- link right_link22: geometry collision mesh filename=/home/xufangjin/workspace/zerograsp/maniskill_curobo_fangzh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; visual mesh filename=/home/xufangjin/workspace/zerograsp/maniskill_curobo_fangzh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
- link right_link23: geometry collision mesh filename=/home/xufangjin/workspace/zerograsp/maniskill_curobo_fangzh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; visual mesh filename=/home/xufangjin/workspace/zerograsp/maniskill_curobo_fangzh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
- link right_link24: geometry collision mesh filename=/home/xufangjin/workspace/zerograsp/maniskill_curobo_fangzh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; visual mesh filename=/home/xufangjin/workspace/zerograsp/maniskill_curobo_fangzh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
- link right_link25: geometry collision mesh filename=/home/xufangjin/workspace/zerograsp/maniskill_curobo_fangzh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; visual mesh filename=/home/xufangjin/workspace/zerograsp/maniskill_curobo_fangzh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
- link right_link26: geometry collision mesh filename=/home/xufangjin/workspace/zerograsp/maniskill_curobo_fangzh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; visual mesh filename=/home/xufangjin/workspace/zerograsp/maniskill_curobo_fangzh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
- link right_link27: geometry collision mesh filename=/home/xufangjin/workspace/zerograsp/maniskill_curobo_fangzh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; visual mesh filename=/home/xufangjin/workspace/zerograsp/maniskill_curobo_fangzh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
- link right_link28: geometry collision mesh filename=/home/xufangjin/workspace/zerograsp/maniskill_curobo_fangzh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; visual mesh filename=/home/xufangjin/workspace/zerograsp/maniskill_curobo_fangzh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
- link wheel1: geometry collision mesh filename=/home/xufangjin/workspace/zerograsp/maniskill_curobo_fangzh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; visual mesh filename=/home/xufangjin/workspace/zerograsp/maniskill_curobo_fangzh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
- link wheel2: geometry collision mesh filename=/home/xufangjin/workspace/zerograsp/maniskill_curobo_fangzh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; visual mesh filename=/home/xufangjin/workspace/zerograsp/maniskill_curobo_fangzh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
- link wheel3: geometry collision mesh filename=/home/xufangjin/workspace/zerograsp/maniskill_curobo_fangzh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; visual mesh filename=/home/xufangjin/workspace/zerograsp/maniskill_curobo_fangzh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

File: maniskill_curobo_fangzhou/generated/lift2_maniskill_visual.urdf (robot description, URDF)
Before this commit: robot lift2, 22 links, 21 joints
Links:
- link base_link: geometry visual mesh filename=/home/xufangjin/workspace/zerograsp/maniskill_curobo_fangzh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
- link body4: geometry visual mesh filename=/home/xufangjin/workspace/zerograsp/maniskill_curobo_fangzh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
- link left_link11: geometry visual mesh filename=/home/xufangjin/workspace/zerograsp/maniskill_curobo_fangzh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
- link left_link12: geometry visual mesh filename=/home/xufangjin/workspace/zerograsp/maniskill_curobo_fangzh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
- link left_link13: geometry visual mesh filename=/home/xufangjin/workspace/zerograsp/maniskill_curobo_fangzh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
- link left_link14: geometry visual mesh filename=/home/xufangjin/workspace/zerograsp/maniskill_curobo_fangzh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
- link left_link15: geometry visual mesh filename=/home/xufangjin/workspace/zerograsp/maniskill_curobo_fangzh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
- link left_link16: geometry visual mesh filename=/home/xufangjin/workspace/zerograsp/maniskill_curobo_fangzh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
- link left_link17: geometry visual mesh filename=/home/xufangjin/workspace/zerograsp/maniskill_curobo_fangzh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
- link left_link18: geometry visual mesh filename=/home/xufangjin/workspace/zerograsp/maniskill_curobo_fangzh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
- link right_link21: geometry visual mesh filename=/home/xufangjin/workspace/zerograsp/maniskill_curobo_fangzh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
- link right_link22: geometry visual mesh filename=/home/xufangjin/workspace/zerograsp/maniskill_curobo_fangzh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
- link right_link23: geometry visual mesh filename=/home/xufangjin/workspace/zerograsp/maniskill_curobo_fangzh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
- link right_link24: geometry visual mesh filename=/home/xufangjin/workspace/zerograsp/maniskill_curobo_fangzh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
- link right_link25: geometry visual mesh filename=/home/xufangjin/workspace/zerograsp/maniskill_curobo_fangzh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
- link right_link26: geometry visual mesh filename=/home/xufangjin/workspace/zerograsp/maniskill_curobo_fangzh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
- link right_link27: geometry visual mesh filename=/home/xufangjin/workspace/zerograsp/maniskill_curobo_fangzh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
- link right_link28: geometry visual mesh filename=/home/xufangjin/workspace/zerograsp/maniskill_curobo_fangzh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
- link wheel1: geometry visual mesh filename=/home/xufangjin/workspace/zerograsp/maniskill_curobo_fangzh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
- link wheel2: geometry visual mesh filename=/home/xufangjin/workspace/zerograsp/maniskill_curobo_fangzh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
- link wheel3: geometry visual mesh filename=/home/xufangjin/workspace/zerograsp/maniskill_curobo_fangzh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
